File: KiCad/ardWatch/ardWatch.kicad_sch (KiCad schematic)
At the start: 4 parts, among them U3 ST7735_1.8"_TFT_128x160, U4 DS3231_RTC_module

Commit message: pcb
Parts:
- added BZ1: (no value), symbol Device:Buzzer
- added U2: (no value), symbol My_Parts:KY-040_Rotary_Encoder
- J1: value (none) -> 2-pin_power_input_header; footprint (none) -> My_Headers:2-pin_power_input_header_larger_pads
- U1: value (none) -> Arduino_Mini_Pro; footprint (none) -> My_Arduino:Arduino_Pro_Mini_vC_larger_pads
Connections:
- net +5V: now also U2.4 (VCC)
- net GND: now also BZ1.2 (+), U2.5 (GND)
- net at U1.10 (7): now also U2.2 (DT)
- net at U1.11 (8): now also U2.1 (CLK)
- net at U1.12 (9): now also BZ1.1 (-)
- net at U1.9 (6): now also U2.3 (SW)
Other:
- moved on the sheet: J1
