File: KiCad/espWatch-ESP01/espWatch-ESP01.kicad_sch (KiCad schematic)
At the start: 10 parts, among them J1 2-pin_power_input_header, SW1 SW_Push, U1 AMS1117-3.3, U2 ESP-01, U3 SSD1306_I2C_display, U4 DS3231_RTC_module

Commit message: better pcb
Parts:
- C1: value 10n -> 100n
Other:
- moved on the sheet: J1, U1
