File: KiCad/espWatch-ESP01/espWatch-ESP01.kicad_pcb (KiCad board)
At the start: 2 copper layers, 55.2 x 41.9 mm, 10 parts, among them J1 2-pin_power_input_header, SW1 SW_Push, U1 AMS1117-3.3, U2 ESP-01, U3 SSD1306_I2C_display, U4 DS3231_RTC_module

Commit message: esp01 pcb
Routing:
- net GND: track 164.5 -> 161.7 mm
- net SCL: track 75.8 -> 74.0 mm
- net SDA: track 67.2 -> 65.7 mm
- net VCC: track 31.5 -> 30.6 mm
- added copper zone on B.Cu, net (none)
- added copper zone on B.Cu, net GND

Commit message: better pcb
Routing:
- net +3V3: track 160.1 -> 141.9 mm
- net GND: track 161.7 -> 156.8 mm, vias 4 -> 2
