File: KiCad/ardWatch-miniPro328/ardWatch-miniPro328.kicad_pcb (KiCad board)
At the start: 2 copper layers, 84.5 x 65.4 mm, 7 parts, among them J1 2-pin_power_input_header, U1 Arduino_Mini_Pro, U2 KY-040_Rotary_Encoder, U3 ST7735_1.8"_TFT_128x160, U4 DS3231_RTC_module

Commit message: schematics
Parts:
- U1: footprint My_Arduino:Arduino_Pro_Mini_vA -> My_Arduino:Arduino_Pro_Mini_vA_sides_n_A4,A5_large
Routing:
- net +5V: track 152.3 -> 158.7 mm
- net Net-(U1-Pad11): track 33.2 -> 34.0 mm
- net Net-(U1-Pad12): track 22.3 -> 21.6 mm

Commit message: revised pcb
Parts:
- J1: footprint My_Headers:2-pin_power_input_header_larger_pads -> My_Headers:2-pin_power_input_header
- moved U4 3.24 mm to (127.6, 99.1)
- moved U2 0.50 mm to (133.3, 103.5)
Connections:
- U3 pad 1: Net-(RV1-Pad2) -> GND
- U3 pad 2: Net-(U1-Pad6) -> +5V
- U3 pad 3: Net-(U1-Pad7) -> Net-(U1-Pad21)
- U3 pad 4: Net-(U1-Pad8) -> Net-(U1-Pad23)
- U3 pad 5: Net-(U1-Pad23) -> Net-(U1-Pad8)
- U3 pad 6: Net-(U1-Pad21) -> Net-(U1-Pad7)
- U3 pad 7: +5V -> Net-(U1-Pad6)
- U3 pad 8: GND -> Net-(RV1-Pad2)
Routing:
- net GND: track 221.5 -> 276.2 mm, vias 2 -> 4
- net VCC: track 25.8 -> 20.3 mm
- net Net-(U1-Pad6): track 148.3 -> 153.1 mm
- net Net-(U1-Pad7): track 140.7 -> 144.1 mm
- net Net-(U1-Pad21): track 30.7 -> 34.1 mm
- net SCL: track 37.4 -> 39.4 mm
- net Net-(U1-Pad8): track 133.2 -> 135.1 mm
- net SDA: track 39.2 -> 37.4 mm, vias 2 -> 0
- net Net-(U1-Pad23): track 37.2 -> 38.6 mm
- net +5V: track 158.7 -> 157.5 mm, vias 0 -> 2
- net Net-(BZ1-Pad1): track 88.5 -> 89.6 mm
Other:
- board size 84.5 x 65.4 mm -> 85.1 x 67.3 mm
- board text added: "5V"
- board text removed: "SDA"

Commit message: new 328 pcb
Parts:
- added R1: R, My_Misc:R_Axial_DIN0207_L6.3mm_D2.5mm_P10.16mm_Horizontal_larger_pads, F.Cu at (145.4, 71.8)
Connections:
- U1 pad 8: Net-(U1-Pad8) -> unconnected-(U1-Pad8)
- U3 pad 5: Net-(U1-Pad8) -> Net-(U3-Pad5)
Routing:
- net Net-(U1-Pad8): track 135.1 -> 0.00 mm
- net Net-(U3-Pad5): track 0.00 -> 57.1 mm
- net GND: track 276.2 -> 314.6 mm
- net +5V: track 157.5 -> 169.2 mm
- net SDA: track 37.4 -> 32.6 mm
- net SCL: track 39.4 -> 37.5 mm
- net Net-(U3-Pad6): track 144.1 -> 143.0 mm
- net Net-(U1-Pad21): track 34.1 -> 34.8 mm
- net Net-(U1-Pad23): track 38.6 -> 39.2 mm
- net Net-(U3-Pad7): track 153.1 -> 152.4 mm

Commit message: new layout
Parts:
- R1: value R -> 10k
Connections:
- net Net-(BZ1-Pad1) renamed BUZ
- net Net-(U1-Pad10) renamed SW
- net Net-(U1-Pad11) renamed DT
- net Net-(U1-Pad12) renamed CLK
- net Net-(U1-Pad21) renamed SCL SCR
- net Net-(U1-Pad23) renamed SDA SCR
- net Net-(U3-Pad6) renamed DC
- net Net-(U3-Pad7) renamed CS
- net SCL renamed SCL RTC
- net SDA renamed SDA RTC
- U1 pad 14: unconnected-(U1-Pad14) -> GND
Routing:
- net GND: track 314.6 -> 331.5 mm
