File: KiCad/ardWatch-miniPro328/ardWatch-miniPro328.kicad_sch (KiCad schematic)
At the start: 7 parts, among them J1 2-pin_power_input_header, U1 Arduino_Mini_Pro, U2 KY-040_Rotary_Encoder, U3 ST7735_1.8"_TFT_128x160, U4 DS3231_RTC_module

Commit message: schematics
Other:
- moved on the sheet: J1, U4
Changed lines of the file:
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@@
   (junction (at 73.66 46.99) (diameter 0) (color 0 0 0 0)
   )
-  (wire (pts (xy 259.08 100.33) (xy 259.08 105.41))
-    (stroke (width 0) (type default) (color 0 0 0 0))
-  )
-  (wire (pts (xy 256.54 97.79) (xy 259.08 97.79))
+  (wire (pts (xy 250.19 92.71) (xy 250.19 97.79))
+    (stroke (width 0) (type default) (color 0 0 0 0))
+  )
+  (wire (pts (xy 247.65 90.17) (xy 250.19 90.17))
     (stroke (width 0) (type default) (color 0 0 0 0))
   )
@@
     (stroke (width 0) (type default) (color 0 0 0 0))
   )
-  (wire (pts (xy 236.22 55.88) (xy 250.19 55.88))
+  (wire (pts (xy 227.33 44.45) (xy 241.3 44.45))
     (stroke (width 0) (type default) (color 0 0 0 0))
   )
@@
     (stroke (width 0) (type default) (color 0 0 0 0))
   )
-  (wire (pts (xy 247.65 50.8) (xy 247.65 43.18))
+  (wire (pts (xy 238.76 39.37) (xy 238.76 31.75))
     (stroke (width 0) (type default) (color 0 0 0 0))
   )
@@
     (stroke (width 0) (type default) (color 0 0 0 0))
   )
-  (wire (pts (xy 250.19 50.8) (xy 247.65 50.8))
+  (wire (pts (xy 241.3 39.37) (xy 238.76 39.37))
     (stroke (width 0) (type default) (color 0 0 0 0))
   )
@@
     (stroke (width 0) (type default) (color 0 0 0 0))
   )
-  (wire (pts (xy 259.08 97.79) (xy 259.08 92.71))
+  (wire (pts (xy 250.19 90.17) (xy 250.19 85.09))
     (stroke (width 0) (type default) (color 0 0 0 0))
   )
@@
     (stroke (width 0) (type default) (color 0 0 0 0))
   )
-  (wire (pts (xy 247.65 68.58) (xy 247.65 60.96))
+  (wire (pts (xy 238.76 57.15) (xy 238.76 49.53))
     (stroke (width 0) (type default) (color 0 0 0 0))
   )
@@
     (stroke (width 0) (type default) (color 0 0 0 0))
   )
-  (wire (pts (xy 247.65 60.96) (xy 250.19 60.96))
-    (stroke (width 0) (type default) (color 0 0 0 0))
-  )
-  (wire (pts (xy 245.11 53.34) (xy 250.19 53.34))
+  (wire (pts (xy 238.76 49.53) (xy 241.3 49.53))
+    (stroke (width 0) (type default) (color 0 0 0 0))
+  )
+  (wire (pts (xy 236.22 41.91) (xy 241.3 41.91))
     (stroke (width 0) (type default) (color 0 0 0 0))
   )
@@
     (stroke (width 0) (type default) (color 0 0 0 0))
   )
-  (wire (pts (xy 256.54 100.33) (xy 259.08 100.33))
+  (wire (pts (xy 247.65 92.71) (xy 250.19 92.71))
     (stroke (width 0) (type default) (color 0 0 0 0))
   )
@@
     )
   )
-  (global_label "SCL" (shape input) (at 236.22 55.88 180) (fields_autoplaced)
+  (global_label "SCL" (shape input) (at 227.33 44.45 180) (fields_autoplaced)
     (effects (font (size 1.27 1.27)) (justify right))
-    (property "Intersheet References" "${INTERSHEET_REFS}" (id 0) (at 230.2993 55.8006 0)
+    (property "Intersheet References" "${INTERSHEET_REFS}" (id 0) (at 221.4093 44.3706 0)
       (effects (font (size 1.27 1.27)) (justify right) hide)
     )
   )
-  (global_label "SDA" (shape input) (at 245.11 53.34 180) (fields_autoplaced)
+  (global_label "SDA" (shape input) (at 236.22 41.91 180) (fields_autoplaced)
     (effects (font (size 1.27 1.27)) (justify right))
-    (property "Intersheet References" "${INTERSHEET_REFS}" (id 0) (at 239.1288 53.2606 0)
+    (property "Intersheet References" "${INTERSHEET_REFS}" (id 0) (at 230.2388 41.8306 0)
       (effects (font (size 1.27 1.27)) (justify right) hide)
     )
@@
     (pin "5")
   )
-  (symbol (lib_id "power:VCC") (at 259.08 92.71 0) (unit 1)
-    (in_bom yes) (on_board yes) (fields_autoplaced)
-    (property "Reference" "#PWR0107" (id 0) (at 259.08 96.52 0)
-      (effects (font (size 1.27 1.27)) hide)
-    )
-    (property "Value" "VCC" (id 1) (at 259.08 89.1342 0))
-    (property "Footprint" "" (id 2) (at 259.08 92.71 0)
-      (effects (font (size 1.27 1.27)) hide)
-    )
-    (property "Datasheet" "" (id 3) (at 259.08 92.71 0)
+  (symbol (lib_id "power:VCC") (at 250.19 85.09 0) (unit 1)
+    (in_bom yes) (on_board yes) (fields_autoplaced)
+    (property "Reference" "#PWR0107" (id 0) (at 250.19 88.9 0)
+      (effects (font (size 1.27 1.27)) hide)
+    )
+    (property "Value" "VCC" (id 1) (at 250.19 81.5142 0))
+    (property "Footprint" "" (id 2) (at 250.19 85.09 0)
+      (effects (font (size 1.27 1.27)) hide)
+    )
+    (property "Datasheet" "" (id 3) (at 250.19 85.09 0)
       (effects (font (size 1.27 1.27)) hide)
     )
@@
     (pin "2")
   )
-  (symbol (lib_id "power:GND") (at 259.08 105.41 0) (unit 1)
-    (in_bom yes) (on_board yes) (fields_autoplaced)
-    (property "Reference" "#PWR0108" (id 0) (at 259.08 111.76 0)
-      (effects (font (size 1.27 1.27)) hide)
-    )
-    (property "Value" "GND" (id 1) (at 259.08 109.8534 0))
-    (property "Footprint" "" (id 2) (at 259.08 105.41 0)
-      (effects (font (size 1.27 1.27)) hide)
-    )
-    (property "Datasheet" "" (id 3) (at 259.08 105.41 0)
+  (symbol (lib_id "power:GND") (at 250.19 97.79 0) (unit 1)
+    (in_bom yes) (on_board yes) (fields_autoplaced)
+    (property "Reference" "#PWR0108" (id 0) (at 250.19 104.14 0)
+      (effects (font (size 1.27 1.27)) hide)
+    )
+    (property "Value" "GND" (id 1) (at 250.19 102.2334 0))
+    (property "Footprint" "" (id 2) (at 250.19 97.79 0)
+      (effects (font (size 1.27 1.27)) hide)
+    )
+    (property "Datasheet" "" (id 3) (at 250.19 97.79 0)
       (effects (font (size 1.27 1.27)) hide)
     )
@@
     (pin "1")
   )
-  (symbol (lib_id "power:GND") (at 247.65 68.58 0) (unit 1)
-    (in_bom yes) (on_board yes) (fields_autoplaced)
-    (property "Reference" "#PWR0102" (id 0) (at 247.65 74.93 0)
-      (effects (font (size 1.27 1.27)) hide)
-    )
-    (property "Value" "GND" (id 1) (at 247.65 73.0234 0))
-    (property "Footprint" "" (id 2) (at 247.65 68.58 0)
-      (effects (font (size 1.27 1.27)) hide)
-    )
-    (property "Datasheet" "" (id 3) (at 247.65 68.58 0)
-      (effects (font (size 1.27 1.27)) hide)
-    )
-    (pin "1")
-  )
-  (symbol (lib_id "My_Headers:2-pin_power_input_header") (at 251.46 97.79 0) (mirror y) (unit 1)
-    (in_bom yes) (on_board yes) (fields_autoplaced)
-    (property "Reference" "J1" (id 0) (at 252.095 96.17 0))
-    (property "Value" "2-pin_power_input_header" (id 1) (at 251.46 102.87 0)
-      (effects (font (size 1.27 1.27)) hide)
-    )
-    (property "Footprint" "My_Headers:2-pin_power_input_header_larger_pads" (id 2) (at 250.19 105.41 0)
-      (effects (font (size 1.27 1.27)) hide)
-    )
-    (property "Datasheet" "~" (id 3) (at 251.46 97.79 0)
+  (symbol (lib_id "power:GND") (at 238.76 57.15 0) (unit 1)
+    (in_bom yes) (on_board yes) (fields_autoplaced)
+    (property "Reference" "#PWR0102" (id 0) (at 238.76 63.5 0)
+      (effects (font (size 1.27 1.27)) hide)
+    )
+    (property "Value" "GND" (id 1) (at 238.76 61.5934 0))
+    (property "Footprint" "" (id 2) (at 238.76 57.15 0)
+      (effects (font (size 1.27 1.27)) hide)
+    )
+    (property "Datasheet" "" (id 3) (at 238.76 57.15 0)
+      (effects (font (size 1.27 1.27)) hide)
+    )
+    (pin "1")
+  )
+  (symbol (lib_id "My_Headers:2-pin_power_input_header") (at 242.57 90.17 0) (mirror y) (unit 1)
+    (in_bom yes) (on_board yes) (fields_autoplaced)
+    (property "Reference" "J1" (id 0) (at 243.205 88.55 0))
+    (property "Value" "2-pin_power_input_header" (id 1) (at 242.57 95.25 0)
+      (effects (font (size 1.27 1.27)) hide)
+    )
+    (property "Footprint" "My_Headers:2-pin_power_input_header_larger_pads" (id 2) (at 241.3 97.79 0)
+      (effects (font (size 1.27 1.27)) hide)
+    )
+    (property "Datasheet" "~" (id 3) (at 242.57 90.17 0)
       (effects (font (size 1.27 1.27)) hide)
     )
@@
     (pin "1")
   )
-  (symbol (lib_id "power:+5V") (at 247.65 43.18 0) (unit 1)
-    (in_bom yes) (on_board yes) (fields_autoplaced)
-    (property "Reference" "#PWR0104" (id 0) (at 247.65 46.99 0)
-      (effects (font (size 1.27 1.27)) hide)
-    )
-    (property "Value" "+5V" (id 1) (at 247.65 39.6042 0))
-    (property "Footprint" "" (id 2) (at 247.65 43.18 0)
-      (effects (font (size 1.27 1.27)) hide)
-    )
-    (property "Datasheet" "" (id 3) (at 247.65 43.18 0)
-      (effects (font (size 1.27 1.27)) hide)
-    )
-    (pin "1")
-  )
-  (symbol (lib_id "My_Parts:DS3231_RTC_module") (at 250.19 50.8 0) (unit 1)
-    (in_bom yes) (on_board yes) (fields_autoplaced)
-    (property "Reference" "U4" (id 0) (at 266.7762 55.0453 0)
+  (symbol (lib_id "power:+5V") (at 238.76 31.75 0) (unit 1)
+    (in_bom yes) (on_board yes) (fields_autoplaced)
+    (property "Reference" "#PWR0104" (id 0) (at 238.76 35.56 0)
+      (effects (font (size 1.27 1.27)) hide)
+    )
+    (property "Value" "+5V" (id 1) (at 238.76 28.1742 0))
+    (property "Footprint" "" (id 2) (at 238.76 31.75 0)
+      (effects (font (size 1.27 1.27)) hide)
+    )
+    (property "Datasheet" "" (id 3) (at 238.76 31.75 0)
+      (effects (font (size 1.27 1.27)) hide)
+    )
+    (pin "1")
+  )
+  (symbol (lib_id "My_Parts:DS3231_RTC_module") (at 241.3 39.37 0) (unit 1)
+    (in_bom yes) (on_board yes) (fields_autoplaced)
+    (property "Reference" "U4" (id 0) (at 257.8862 43.6153 0)
       (effects (font (size 1.27 1.27)) (justify left))
     )
-    (property "Value" "DS3231_RTC_module" (id 1) (at 266.7762 57.5822 0)
+    (property "Value" "DS3231_RTC_module" (id 1) (at 257.8862 46.1522 0)
       (effects (font (size 1.27 1.27)) (justify left))
     )
-    (property "Footprint" "My_Parts:DS3231_RTC_module_large" (id 2) (at 250.19 50.8 0)
-      (effects (font (size 1.27 1.27)) hide)
-    )
-    (property "Datasheet" "" (id 3) (at 250.19 50.8 0)
+    (property "Footprint" "My_Parts:DS3231_RTC_module_large" (id 2) (at 241.3 39.37 0)
+      (effects (font (size 1.27 1.27)) hide)
+    )
+    (property "Datasheet" "" (id 3) (at 241.3 39.37 0)
       (effects (font (size 1.27 1.27)) hide)
     )
@@
     )
     (path "/10d1167f-ef8a-4476-b647-4bb4b8023bd2"
-      (reference "U1") (unit 1) (value "Arduino_Mini_Pro") (footprint "My_Arduino:Arduino_Pro_Mini_vA")
+      (reference "U1") (unit 1) (value "Arduino_Mini_Pro") (footprint "My_Arduino:Arduino_Pro_Mini_vA_sides_n_A4,A5_large")
     )
     (path "/53d31753-c544-4e13-9554-351e472e84f3"

Commit message: revised pcb
Parts:
- J1: footprint My_Headers:2-pin_power_input_header_larger_pads -> My_Headers:2-pin_power_input_header
- U1: footprint (none) -> My_Arduino:Arduino_Pro_Mini_vA_sides_n_A4,A5_large
Connections:
- net +5V: now also U3.2 (VCC); no longer U3.7 (VCC)
- net GND: now also U3.1 (GND); no longer U3.8 (GND)
- net at U1.21 (13): now also U3.3 (SCL); no longer U3.6 (SCL)
- net at U1.23 (11): now also U3.4 (SDA); no longer U3.5 (SDA)
- net at U1.6 (3): now also U3.7 (CS); no longer U3.2 (CS)
- net at U1.7 (4): now also U3.6 (DC); no longer U3.3 (DC)
- net at U1.8 (5): now also U3.5 (RES); no longer U3.4 (RES)
- net at RV1.2: now also U3.8 (BL); no longer U3.1 (BL)
Changed lines of the file:
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@@
-    (stroke (width 0) (type default) (color 0 0 0 0))
-  )
-  (wire (pts (xy 241.3 39.37) (xy 238.76 39.37))
     (stroke (width 0) (type default) (color 0 0 0 0))
   )
@@
   )
   (wire (pts (xy 204.47 102.87) (xy 194.31 102.87))
+    (stroke (width 0) (type default) (color 0 0 0 0))
+  )
+  (wire (pts (xy 238.76 39.37) (xy 241.3 39.37))
     (stroke (width 0) (type default) (color 0 0 0 0))
   )
@@
       (effects (font (size 1.27 1.27)) (justify left))
     )
-    (property "Footprint" "" (id 2) (at 142.24 91.44 0)
+    (property "Footprint" "My_Arduino:Arduino_Pro_Mini_vA_sides_n_A4,A5_large" (id 2) (at 142.24 91.44 0)
       (effects (font (size 1.27 1.27)) hide)
     )
@@
       (effects (font (size 1.27 1.27)) hide)
     )
-    (property "Footprint" "My_Headers:2-pin_power_input_header_larger_pads" (id 2) (at 241.3 97.79 0)
+    (property "Footprint" "My_Headers:2-pin_power_input_header" (id 2) (at 241.3 97.79 0)
       (effects (font (size 1.27 1.27)) hide)
     )
@@
     (pin "1")
   )
-  (symbol (lib_id "My_Parts:DS3231_RTC_module") (at 241.3 39.37 0) (unit 1)
-    (in_bom yes) (on_board yes) (fields_autoplaced)
-    (property "Reference" "U4" (id 0) (at 257.8862 43.6153 0)
-      (effects (font (size 1.27 1.27)) (justify left))
-    )
-    (property "Value" "DS3231_RTC_module" (id 1) (at 257.8862 46.1522 0)
-      (effects (font (size 1.27 1.27)) (justify left))
-    )
-    (property "Footprint" "My_Parts:DS3231_RTC_module_large" (id 2) (at 241.3 39.37 0)
-      (effects (font (size 1.27 1.27)) hide)
-    )
-    (property "Datasheet" "" (id 3) (at 241.3 39.37 0)
+  (symbol (lib_id "My_Parts:DS3231_RTC_module") (at 241.3 49.53 0) (mirror x) (unit 1)
+    (in_bom yes) (on_board yes) (fields_autoplaced)
+    (property "Reference" "U4" (id 0) (at 251.46 33.816 0))
+    (property "Value" "DS3231_RTC_module" (id 1) (at 251.46 36.3529 0))
+    (property "Footprint" "My_Parts:DS3231_RTC_module_large" (id 2) (at 241.3 49.53 0)
+      (effects (font (size 1.27 1.27)) hide)
+    )
+    (property "Datasheet" "" (id 3) (at 241.3 49.53 0)
       (effects (font (size 1.27 1.27)) hide)
     )
@@
     )
     (path "/cdbb4ebf-e670-485c-acfc-c535f0663dca"
-      (reference "J1") (unit 1) (value "2-pin_power_input_header") (footprint "My_Headers:2-pin_power_input_header_larger_pads")
+      (reference "J1") (unit 1) (value "2-pin_power_input_header") (footprint "My_Headers:2-pin_power_input_header")
     )
     (path "/488f0a8c-afa0-4991-97f4-7c1725dbe36d"

Commit message: new 328 pcb
Parts:
- added R1: (no value), symbol Device:R
Connections:
- net +5V: now also R1.1
- net at U1.8 (5): no longer U3.5 (RES)
- new net: R1.2, U3.5 (RES)
Changed lines of the file:
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@@
-    (stroke (width 0) (type default) (color 0 0 0 0))
-  )
-  (wire (pts (xy 101.6 115.57) (xy 101.6 60.96))
     (stroke (width 0) (type default) (color 0 0 0 0))
   )
@@
     (stroke (width 0) (type default) (color 0 0 0 0))
   )
-  (wire (pts (xy 101.6 60.96) (xy 121.92 60.96))
-    (stroke (width 0) (type default) (color 0 0 0 0))
-  )
   (wire (pts (xy 250.19 90.17) (xy 250.19 85.09))
     (stroke (width 0) (type default) (color 0 0 0 0))
@@
     (stroke (width 0) (type default) (color 0 0 0 0))
   )
-  (wire (pts (xy 71.12 115.57) (xy 101.6 115.57))
-    (stroke (width 0) (type default) (color 0 0 0 0))
-  )
   (wire (pts (xy 106.68 128.27) (xy 177.8 128.27))
     (stroke (width 0) (type default) (color 0 0 0 0))
@@
     (stroke (width 0) (type default) (color 0 0 0 0))
   )
+  (wire (pts (xy 82.55 46.99) (xy 73.66 46.99))
+    (stroke (width 0) (type default) (color 0 0 0 0))
+  )
   (wire (pts (xy 73.66 46.99) (xy 73.66 123.19))
     (stroke (width 0) (type default) (color 0 0 0 0))
@@
     (stroke (width 0) (type default) (color 0 0 0 0))
   )
+  (wire (pts (xy 82.55 115.57) (xy 82.55 102.87))
+    (stroke (width 0) (type default) (color 0 0 0 0))
+  )
   (wire (pts (xy 104.14 63.5) (xy 121.92 63.5))
     (stroke (width 0) (type default) (color 0 0 0 0))
@@
     (stroke (width 0) (type default) (color 0 0 0 0))
   )
+  (wire (pts (xy 71.12 115.57) (xy 82.55 115.57))
+    (stroke (width 0) (type default) (color 0 0 0 0))
+  )
   (wire (pts (xy 201.93 68.58) (xy 175.26 68.58))
     (stroke (width 0) (type default) (color 0 0 0 0))
@@
   )
   (wire (pts (xy 160.02 43.18) (xy 189.23 43.18))
+    (stroke (width 0) (type default) (color 0 0 0 0))
+  )
+  (wire (pts (xy 82.55 95.25) (xy 82.55 46.99))
     (stroke (width 0) (type default) (color 0 0 0 0))
   )
@@
     (pin "1")
   )
+  (symbol (lib_id "Device:R") (at 82.55 99.06 0) (unit 1)
+    (in_bom yes) (on_board yes) (fields_autoplaced)
+    (property "Reference" "R1" (id 0) (at 84.328 98.2253 0)
+      (effects (font (size 1.27 1.27)) (justify left))
+    )
+    (property "Value" "" (id 1) (at 84.328 100.7622 0)
+      (effects (font (size 1.27 1.27)) (justify left))
+    )
+    (property "Footprint" "" (id 2) (at 80.772 99.06 90)
+      (effects (font (size 1.27 1.27)) hide)
+    )
+    (property "Datasheet" "~" (id 3) (at 82.55 99.06 0)
+      (effects (font (size 1.27 1.27)) hide)
+    )
+    (pin "1")
+    (pin "2")
+  )
   (symbol (lib_id "power:+5V") (at 194.31 33.02 0) (unit 1)
     (in_bom yes) (on_board yes) (fields_autoplaced)
@@
       (reference "J1") (unit 1) (value "2-pin_power_input_header") (footprint "My_Headers:2-pin_power_input_header")
     )
+    (path "/6d012fbc-a5e9-4e1f-84d4-e411fd28d128"
+      (reference "R1") (unit 1) (value "R") (footprint "My_Misc:R_Axial_DIN0207_L6.3mm_D2.5mm_P10.16mm_Horizontal_larger_pads")
+    )
     (path "/488f0a8c-afa0-4991-97f4-7c1725dbe36d"

Commit message: new layout
Parts:
- R1: value (none) -> 10k; footprint (none) -> My_Misc:R_Axial_DIN0207_L6.3mm_D2.5mm_P10.16mm_Horizontal_larger_pads
Connections:
- net GND: now also U1.14 (GND)
- net SW: now reaches U1.10 (7), U2.3 (SW)
- net DT: now reaches U1.11 (8), U2.2 (DT)
- net CLK: now reaches U1.12 (9), U2.1 (CLK)
- net SCL SCR: now reaches U1.21 (13), U3.3 (SCL)
- net SDA SCR: now reaches U1.23 (11), U3.4 (SDA)
- net CS: now reaches U1.6 (3), U3.7 (CS)
- net DC: now reaches U1.7 (4), U3.6 (DC)
- net BUZ: now reaches BZ1.1 (-), U1.9 (6)
- net SCL renamed SCL RTC
- net SDA renamed SDA RTC
Other:
- moved on the sheet: BZ1, J1, R1, RV1, U2, U3, U4

Commit message: esp01 minimal
Other:
- moved on the sheet: BZ1, J1, R1, RV1, U2, U3, U4
