File: KiCad/ardWatch-uno/ardWatch-uno.kicad_sch (KiCad schematic)
At the start: 8 parts, among them J1 2-pin_power_input_header, U2 KY-040_Rotary_Encoder, U3 ST7735_1.8"_TFT_128x160, U4 DS3231_RTC_module

Commit message: kicad v8
Parts:
- A1: value (none) -> Arduino_UNO_R3; footprint (none) -> My_Arduino:Arduino_UNO_R3_shield_large
