File: KiCad/espWatch/espWatch.kicad_pcb (KiCad board)
At the start: 2 copper layers, 81.3 x 73 mm, 5 parts, among them U1 Level converter, U2 NodeMCU_1.0_(ESP-12E), U3 1.8" TFT ST7735, U4 RTC DS3231

Commit message: schematics
Parts:
- added RV1: R_Potentiometer, My_Misc:Potentiometer_Bourns_3339P_Vertical_large, F.Cu at (145.4, 60.9)
- moved BZ1 33.2 mm to (117.6, 75.6)
Connections:
- BZ1 pad 1: /Buzz -> Net-(U2-Pad20)
- U2 pad 20: unconnected-(U2-Pad20) -> Net-(U2-Pad20)
- U2 pad 21: unconnected-(U2-Pad21) -> Net-(U2-Pad21)
- U2 pad 22: unconnected-(U2-Pad22) -> Net-(U2-Pad22)
- U2 pad 23: unconnected-(U2-Pad23) -> Net-(U2-Pad23)
- U2 pad 26: unconnected-(U2-Pad26) -> Net-(U3-Pad6)
- U3 pad 1: unconnected-(U3-Pad1) -> GND
- U3 pad 2: unconnected-(U3-Pad2) -> +5V
- U3 pad 3: unconnected-(U3-Pad3) -> Net-(U2-Pad23)
- U3 pad 4: unconnected-(U3-Pad4) -> Net-(U2-Pad21)
- U3 pad 5: /SDA H -> Net-(U2-Pad22)
- U3 pad 6: /SCL H -> Net-(U3-Pad6)
- U3 pad 7: +5V -> /Buzz
- U3 pad 8: GND -> Net-(U3-Pad8)
- U4 pad 2: /SCL H -> /SDA H
- U4 pad 3: /SDA H -> /SCL H
Routing:
- net /Buzz: track 0.00 -> 118.1 mm
- net Net-(U3-Pad6): track 0.00 -> 110.7 mm
- net Net-(U2-Pad22): track 0.00 -> 98.9 mm
- net /SDA H: track 93.2 -> 17.6 mm
- net /SCL H: track 89.7 -> 17.6 mm
- net Net-(U3-Pad8): track 0.00 -> 62.9 mm
- net Net-(U2-Pad21): track 0.00 -> 45.0 mm
- net Net-(U2-Pad23): track 0.00 -> 37.4 mm
- net +5V: track 206.4 -> 184.8 mm, vias 2 -> 0
- net GND: track 204.0 -> 222.5 mm, vias 4 -> 0
- net Net-(U2-Pad20): track 0.00 -> 14.1 mm
- net +3V3: track 78.4 -> 67.2 mm, vias 4 -> 0
- net /SCL L: track 62.6 -> 71.2 mm
- net /SDA L: track 63.1 -> 69.5 mm
Other:
- outline, holes or cut-outs redrawn
- board text removed: "3.3V"
- board text removed: "5V"
- board text removed: "GND"

Commit message: nodemcu
Parts:
- moved RV1 0.10 mm to (145.3, 60.9)
Connections:
- RV1 pad 3: +5V -> +3V3
- U3 pad 2: +5V -> +3V3
Routing:
- net +3V3: track 67.2 -> 229.9 mm, vias 0 -> 2
- net +5V: track 184.8 -> 69.6 mm, vias 0 -> 2
- net GND: track 222.5 -> 266.1 mm, vias 0 -> 4
- net /Buzz: track 118.1 -> 133.9 mm
- net /SCL L: track 71.2 -> 64.4 mm
- net /SDA L: track 69.5 -> 63.7 mm
- net Net-(U2-Pad26): track 110.7 -> 115.3 mm
- net Net-(U2-Pad23): track 37.4 -> 41.0 mm
- net Net-(U2-Pad22): track 98.9 -> 100.6 mm
- net Net-(U2-Pad21): track 45.0 -> 46.3 mm
- net Net-(RV1-Pad2): track 62.9 -> 62.1 mm
- added copper zone on B.Cu, net (none)
- added copper zone on B.Cu, net GND
Other:
- board size 81.3 x 73 mm -> 82.6 x 73.7 mm
- board text added: "3.3V"
- board text added: "5V"
- board text added: "GND"

Commit message: pcb and pin config
Parts:
- removed U1: Level converter, My_Parts:4-channel_I2C_level_shifter_BSS138_large
- added R1: 10k, My_Misc:R_Axial_DIN0207_L6.3mm_D2.5mm_P10.16mm_Horizontal_larger_pads, F.Cu at (101.6, 76.2)
- added U5: KY-040_Rotary_Encoder, My_Parts:KY-040_rotary_encoder module_w_header_large, F.Cu at (161.9, 76.2)
- moved U4 21.0 mm to (149.9, 109.9), turned to 180 degrees
Connections:
- net /Buzz renamed Net-(U2-Pad27)
- U2 pad 22: Net-(U2-Pad22) -> unconnected-(U2-Pad22)
- U2 pad 30: unconnected-(U2-Pad30) -> Net-(U2-Pad30)
- U2 pad 4: unconnected-(U2-Pad4) -> Net-(U5-Pad1)
- U2 pad 5: unconnected-(U2-Pad5) -> Net-(U5-Pad2)
- U3 pad 5: Net-(U2-Pad22) -> Net-(U3-Pad5)
- U4 pad 1: +5V -> +3V3
- U4 pad 2: /SDA H -> /SDA L
- U4 pad 3: /SCL H -> /SCL L
Routing:
- net Net-(U2-Pad30): track 0.00 -> 156.8 mm
- net Net-(U5-Pad1): track 0.00 -> 113.9 mm
- net Net-(U5-Pad2): track 0.00 -> 104.5 mm
- net Net-(U2-Pad22): track 100.6 -> 0.00 mm
- net +5V: track 69.6 -> 0.00 mm, vias 2 -> 0
- net GND: track 266.1 -> 317.3 mm, vias 4 -> 2
- net +3V3: track 229.9 -> 274.2 mm
- net Net-(U3-Pad5): track 0.00 -> 21.6 mm
- net /SDA H: track 17.8 -> 0.00 mm
- net Net-(U2-Pad27): track 133.9 -> 116.3 mm
- net /SCL H: track 17.1 -> 0.00 mm
- net Net-(U2-Pad26): track 115.3 -> 105.7 mm
- net /SCL L: track 64.4 -> 66.5 mm
- net Net-(U2-Pad23): track 41.0 -> 39.4 mm
- net Net-(U2-Pad21): track 46.3 -> 45.0 mm
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Other:
- board size 82.6 x 73.7 mm -> 96.5 x 79.4 mm
- board text added: "3V3"
- board text removed: "3.3V"
- board text removed: "5V"

Commit message: moverd rtc
Parts:
- moved U4 6.48 mm to (156.2, 108.6)
Routing:
- net GND: track 317.3 -> 286.2 mm
- net /SCL L: track 66.5 -> 74.9 mm
- net /SDA L: track 63.8 -> 71.2 mm
- net +3V3: track 274.2 -> 272.7 mm

Commit message: added power input header
Parts:
- added J1: 2-pin_power_input_header, My_Headers:2-pin_power_input_header_larger_pads, F.Cu at (140.3, 112.4)
Routing:
- net +5V: track 0.00 -> 17.5 mm
- net GND: track 286.2 -> 291.3 mm

Commit message: new schematics for esp
Connections:
- net /SCL L renamed SCL RTC
- net /SDA L renamed SDA RTC
- net Net-(BZ1-Pad1) renamed BUZ
- net Net-(U2-Pad21) renamed SDA SCR
- net Net-(U2-Pad23) renamed SCL SCR
- net Net-(U2-Pad26) renamed DC
- net Net-(U2-Pad27) renamed CS
- net Net-(U2-Pad30) renamed SW
- net Net-(U2-Pad4) renamed CLK
- net Net-(U2-Pad5) renamed DT

Commit message: new pcb
Parts:
- moved U3 104.4 mm to (169.5, 112.3), turned to 180 degrees
- moved U2 89.3 mm to (151.0, 52.7), turned to -90 degrees
- moved RV1 64.4 mm to (109.3, 114.3)
- moved J1 42.7 mm to (106.0, 87.0)
- moved U4 39.5 mm to (177.5, 75.3), turned to 0 degrees
- moved R1 35.1 mm to (121.9, 104.8), turned to 0 degrees
- moved U5 34.0 mm to (188.4, 54.8)
- moved BZ1 26.2 mm to (134.2, 95.9)
Connections:
- RV1 pad 1: GND -> +3V3
- RV1 pad 3: +3V3 -> GND
Routing:
- net SW: track 156.8 -> 49.4 mm
- net CLK: track 113.9 -> 48.5 mm
- net DT: track 104.5 -> 52.4 mm
- net SCL RTC: track 74.9 -> 30.1 mm
- net SDA RTC: track 71.2 -> 34.6 mm
- net GND: track 291.3 -> 259.1 mm, vias 2 -> 4
- net +3V3: track 272.7 -> 298.2 mm, vias 2 -> 0
- net +5V: track 17.5 -> 38.4 mm
- net Net-(R1-Pad2): track 21.6 -> 38.1 mm
- net CS: track 116.3 -> 132.7 mm
- net DC: track 105.7 -> 121.8 mm
- net Net-(RV1-Pad2): track 62.8 -> 72.2 mm
- net SCL SCR: track 39.4 -> 45.6 mm
- net SDA SCR: track 45.0 -> 50.3 mm
- net BUZ: track 15.0 -> 18.5 mm
Other:
- board size 96.5 x 79.4 mm -> 92.7 x 74.3 mm
- board text added: "espWatch Design: Jon Sagebrand github.com/jonsag/mcuWatch"
- board text removed: "3V3"
- board text removed: "Design: Jon Sagebrand jonsagebrand@gmail.com github.com/jonsag/mcuWatch"
- board text removed: "Design: Jon Sagebrand mcuWatch github.com/jonsag"
