File: KiCad/espWatch/espWatch.kicad_sch (KiCad schematic)
At the start: 5 parts, among them U2 NodeMCU_1.0_(ESP-12E)

Commit message: schematics
Parts:
- added RV1: (no value), symbol Device:R_Potentiometer
- BZ1: value (none) -> Buzzer; footprint (none) -> My_Misc:Buzzer_TDK_PS1240P02BT_D12.2mm_H6.5mm_large
- U1: value (none) -> Level converter
- U3: value (none) -> 1.8" TFT ST7735
- U4: value (none) -> RTC DS3231
Connections:
- net +5V: now also U3.2 (VCC), RV1.3; no longer U3.7 (VCC)
- net Buzz: now also U3.7 (CS); no longer BZ1.1 (-)
- net GND: now also U3.1 (GND), RV1.1; no longer U3.8 (GND)
- net SCL H: now also U4.3 (C_SCL); no longer U3.6 (SCL), U4.2 (D_SDA)
- net SDA H: now also U4.2 (D_SDA); no longer U3.5 (SDA), U4.3 (C_SCL)
- net at U2.20 (D8(GPIO15)): now also BZ1.1 (-)
- net at U2.21 (D7(GPIO13)): now also U3.4 (SDA)
- net at U2.22 (D6(GPIO12)): now also U3.5 (RES)
- net at U2.23 (D5(GPIO14)): now also U3.3 (SCL)
- net at U2.26 (D4(GPIO2)): now also U3.6 (DC)
- new net: RV1.2, U3.8 (BL)
Other:
- moved on the sheet: BZ1, U3, U4

Commit message: nodemcu
Parts:
- RV1: value (none) -> R_Potentiometer; footprint (none) -> My_Misc:Potentiometer_Bourns_3339P_Vertical_large
Connections:
- net +3V3: now also RV1.3, U3.2 (VCC)
- net +5V: no longer RV1.3, U3.2 (VCC)
Changed lines of the file:
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@@
       (effects (font (size 1.27 1.27)) (justify right))
     )
-    (property "Value" "" (id 1) (at 99.8221 107.1122 0)
+    (property "Value" "R_Potentiometer" (id 1) (at 99.8221 107.1122 0)
       (effects (font (size 1.27 1.27)) (justify right))
     )
-    (property "Footprint" "" (id 2) (at 101.6 105.41 0)
+    (property "Footprint" "My_Misc:Potentiometer_Bourns_3339P_Vertical_large" (id 2) (at 101.6 105.41 0)
       (effects (font (size 1.27 1.27)) hide)
     )
@@
       (effects (font (size 1.27 1.27)) hide)
     )
-    (property "Value" "" (id 1) (at 101.6 132.7134 0))
+    (property "Value" "GND" (id 1) (at 101.6 132.7134 0))
     (property "Footprint" "" (id 2) (at 101.6 128.27 0)
       (effects (font (size 1.27 1.27)) hide)
@@
     (pin "1")
   )
+  (symbol (lib_id "power:+3.3V") (at 135.89 95.25 0) (unit 1)
+    (in_bom yes) (on_board yes) (fields_autoplaced)
+    (property "Reference" "#PWR?" (id 0) (at 135.89 99.06 0)
+      (effects (font (size 1.27 1.27)) hide)
+    )
+    (property "Value" "" (id 1) (at 135.89 91.6742 0))
+    (property "Footprint" "" (id 2) (at 135.89 95.25 0)
+      (effects (font (size 1.27 1.27)) hide)
+    )
+    (property "Datasheet" "" (id 3) (at 135.89 95.25 0)
+      (effects (font (size 1.27 1.27)) hide)
+    )
+    (pin "1")
+  )
   (symbol (lib_id "power:+3.3V") (at 82.55 29.21 0) (unit 1)
     (in_bom yes) (on_board yes) (fields_autoplaced)
@@
     )
     (property "Datasheet" "" (id 3) (at 201.93 69.85 0)
-      (effects (font (size 1.27 1.27)) hide)
-    )
-    (pin "1")
-  )
-  (symbol (lib_id "power:+5V") (at 135.89 95.25 0) (unit 1)
-    (in_bom yes) (on_board yes)
-    (property "Reference" "#PWR0101" (id 0) (at 135.89 99.06 0)
-      (effects (font (size 1.27 1.27)) hide)
-    )
-    (property "Value" "+5V" (id 1) (at 135.89 91.6742 0))
-    (property "Footprint" "" (id 2) (at 135.89 95.25 0)
-      (effects (font (size 1.27 1.27)) hide)
-    )
-    (property "Datasheet" "" (id 3) (at 135.89 95.25 0)
       (effects (font (size 1.27 1.27)) hide)
     )
@@
   )
   (symbol_instances
-    (path "/d9e401b8-baf3-4ffb-94cf-ae614cfb9092"
-      (reference "#PWR0101") (unit 1) (value "+5V") (footprint "")
-    )
     (path "/cb98afaf-57c8-4a7d-9e8e-3faa1ae4d64d"
       (reference "#PWR0102") (unit 1) (value "GND") (footprint "")
@@
       (reference "#PWR0114") (unit 1) (value "GND") (footprint "")
     )
+    (path "/9396dbf5-aa3c-4ba1-a9ae-1945fbb2026c"
+      (reference "#PWR?") (unit 1) (value "+3.3V") (footprint "")
+    )
     (path "/672233ec-4d06-4b1a-8178-caf57df5342a"

Commit message: pcb and pin config
Parts:
- removed U1: Level converter, My_Parts:4-channel_I2C_level_shifter_BSS138_large, symbol My_Parts:4-channel_I2C_level_shifter_BSS138
- added R1: (no value), symbol Device:R
- added U5: (no value), symbol My_Parts:KY-040_Rotary_Encoder
Connections:
- net SCL H is gone; now on net SCL L: U4.3 (C_SCL)
- net SDA H is gone; now on net SDA L: U4.2 (D_SDA)
- net +3V3: now also U4.1 (VCC), R1.1, U5.4 (VCC)
- net +5V: no longer U4.1 (VCC)
- net GND: now also U5.5 (GND)
- net at U3.5 (RES): now also R1.2; no longer U2.22 (D6(GPIO12))
- net at U2.30 (D0(GPIO16)): now also U5.3 (SW)
- net at U2.4 (SD3(GPIO10)): now also U5.1 (CLK)
- net at U2.5 (SD2(GPIO9)): now also U5.2 (DT)
- net Buzz: no longer names the net of U2.27 (D3(GPIO0)), U3.7 (CS)

Commit message: added power input header
Parts:
- added J1: (no value), symbol My_Headers:2-pin_power_input_header
- R1: value (none) -> 10k; footprint (none) -> My_Misc:R_Axial_DIN0207_L6.3mm_D2.5mm_P10.16mm_Horizontal_larger_pads
- U5: value (none) -> KY-040_Rotary_Encoder; footprint (none) -> My_Parts:KY-040_rotary_encoder module_w_header_large
Connections:
- net +5V: now also J1.1 (VCC)
- net GND: now also J1.2 (GND)
Changed lines of the file:
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@@
+    (stroke (width 0) (type default) (color 0 0 0 0))
+  )
+  (wire (pts (xy 229.87 97.79) (xy 224.79 97.79))
+    (stroke (width 0) (type default) (color 0 0 0 0))
+  )
+  (wire (pts (xy 229.87 100.33) (xy 224.79 100.33))
     (stroke (width 0) (type default) (color 0 0 0 0))
   )
@@
     (stroke (width 0) (type default) (color 0 0 0 0))
   )
+  (wire (pts (xy 224.79 100.33) (xy 224.79 105.41))
+    (stroke (width 0) (type default) (color 0 0 0 0))
+  )
   (wire (pts (xy 36.83 46.99) (xy 26.67 46.99))
     (stroke (width 0) (type default) (color 0 0 0 0))
@@
   )
   (wire (pts (xy 36.83 62.23) (xy 34.29 62.23))
+    (stroke (width 0) (type default) (color 0 0 0 0))
+  )
+  (wire (pts (xy 224.79 97.79) (xy 224.79 92.71))
     (stroke (width 0) (type default) (color 0 0 0 0))
   )
@@
       (effects (font (size 1.27 1.27)) (justify left))
     )
-    (property "Value" "" (id 1) (at 77.978 107.1122 0)
-      (effects (font (size 1.27 1.27)) (justify left))
-    )
-    (property "Footprint" "" (id 2) (at 74.422 105.41 90)
+    (property "Value" "10k" (id 1) (at 77.978 107.1122 0)
+      (effects (font (size 1.27 1.27)) (justify left))
+    )
+    (property "Footprint" "My_Misc:R_Axial_DIN0207_L6.3mm_D2.5mm_P10.16mm_Horizontal_larger_pads" (id 2) (at 74.422 105.41 90)
       (effects (font (size 1.27 1.27)) hide)
     )
@@
       (effects (font (size 1.27 1.27)) (justify left))
     )
-    (property "Value" "" (id 1) (at 147.955 151.13 0)
-      (effects (font (size 1.27 1.27)) hide)
-    )
-    (property "Footprint" "" (id 2) (at 146.685 153.67 0)
+    (property "Value" "KY-040_Rotary_Encoder" (id 1) (at 147.955 151.13 0)
+      (effects (font (size 1.27 1.27)) hide)
+    )
+    (property "Footprint" "My_Parts:KY-040_rotary_encoder module_w_header_large" (id 2) (at 146.685 153.67 0)
       (effects (font (size 1.27 1.27)) hide)
     )
@@
       (effects (font (size 1.27 1.27)) hide)
     )
-    (property "Value" "" (id 1) (at 133.35 180.9734 0))
+    (property "Value" "GND" (id 1) (at 133.35 180.9734 0))
     (property "Footprint" "" (id 2) (at 133.35 176.53 0)
       (effects (font (size 1.27 1.27)) hide)
@@
       (effects (font (size 1.27 1.27)) hide)
     )
-    (property "Value" "" (id 1) (at 135.89 139.9342 0))
+    (property "Value" "+3.3V" (id 1) (at 135.89 139.9342 0))
     (property "Footprint" "" (id 2) (at 135.89 143.51 0)
       (effects (font (size 1.27 1.27)) hide)
@@
     (pin "1")
   )
+  (symbol (lib_id "power:GND") (at 224.79 105.41 0) (unit 1)
+    (in_bom yes) (on_board yes) (fields_autoplaced)
+    (property "Reference" "#PWR0108" (id 0) (at 224.79 111.76 0)
+      (effects (font (size 1.27 1.27)) hide)
+    )
+    (property "Value" "" (id 1) (at 224.79 109.8534 0))
+    (property "Footprint" "" (id 2) (at 224.79 105.41 0)
+      (effects (font (size 1.27 1.27)) hide)
+    )
+    (property "Datasheet" "" (id 3) (at 224.79 105.41 0)
+      (effects (font (size 1.27 1.27)) hide)
+    )
+    (pin "1")
+  )
   (symbol (lib_id "power:+3.3V") (at 201.93 29.21 0) (unit 1)
     (in_bom yes) (on_board yes) (fields_autoplaced)
@@
       (effects (font (size 1.27 1.27)) hide)
     )
-    (property "Value" "" (id 1) (at 201.93 25.6342 0))
+    (property "Value" "+3.3V" (id 1) (at 201.93 25.6342 0))
     (property "Footprint" "" (id 2) (at 201.93 29.21 0)
       (effects (font (size 1.27 1.27)) hide)
@@
     )
     (property "Datasheet" "" (id 3) (at 201.93 69.85 0)
+      (effects (font (size 1.27 1.27)) hide)
+    )
+    (pin "1")
+  )
+  (symbol (lib_id "My_Headers:2-pin_power_input_header") (at 234.95 97.79 0) (unit 1)
+    (in_bom yes) (on_board yes) (fields_autoplaced)
+    (property "Reference" "J1" (id 0) (at 235.6612 99.4938 0)
+      (effects (font (size 1.27 1.27)) (justify left))
+    )
+    (property "Value" "" (id 1) (at 234.95 102.87 0)
+      (effects (font (size 1.27 1.27)) hide)
+    )
+    (property "Footprint" "" (id 2) (at 236.22 105.41 0)
+      (effects (font (size 1.27 1.27)) hide)
+    )
+    (property "Datasheet" "~" (id 3) (at 234.95 97.79 0)
+      (effects (font (size 1.27 1.27)) hide)
+    )
+    (pin "1")
+    (pin "2")
+  )
+  (symbol (lib_id "power:+5V") (at 224.79 92.71 0) (unit 1)
+    (in_bom yes) (on_board yes) (fields_autoplaced)
+    (property "Reference" "#PWR0107" (id 0) (at 224.79 96.52 0)
+      (effects (font (size 1.27 1.27)) hide)
+    )
+    (property "Value" "" (id 1) (at 224.79 89.1342 0))
+    (property "Footprint" "" (id 2) (at 224.79 92.71 0)
+      (effects (font (size 1.27 1.27)) hide)
+    )
+    (property "Datasheet" "" (id 3) (at 224.79 92.71 0)
       (effects (font (size 1.27 1.27)) hide)
     )
@@
       (reference "#PWR0106") (unit 1) (value "+3.3V") (footprint "")
     )
+    (path "/e397848a-7c5f-4dca-a1cb-8dda896b045e"
+      (reference "#PWR0107") (unit 1) (value "+5V") (footprint "")
+    )
+    (path "/aaab055d-e2c8-47ec-bf52-ba6cbf89c068"
+      (reference "#PWR0108") (unit 1) (value "GND") (footprint "")
+    )
     (path "/e7e8ed8d-4df9-4204-93ee-c3c93707dcc6"
       (reference "#PWR0109") (unit 1) (value "GND") (footprint "")
@@
       (reference "BZ1") (unit 1) (value "Buzzer") (footprint "My_Misc:Buzzer_TDK_PS1240P02BT_D12.2mm_H6.5mm_large")
     )
+    (path "/d8249d3a-6081-432d-aa74-a584290619e8"
+      (reference "J1") (unit 1) (value "2-pin_power_input_header") (footprint "My_Headers:2-pin_power_input_header_larger_pads")
+    )
     (path "/0e1e548c-ec74-46cb-aa6e-5e8839149d3f"

Commit message: new schematics for esp
Parts:
- J1: value (none) -> 2-pin_power_input_header; footprint (none) -> My_Headers:2-pin_power_input_header_larger_pads
Connections:
- net BUZ: now reaches BZ1.1 (-), U2.20 (D8(GPIO15))
- net SDA SCR: now reaches U2.21 (D7(GPIO13)), U3.4 (SDA)
- net SCL SCR: now reaches U2.23 (D5(GPIO14)), U3.3 (SCL)
- net DC: now reaches U2.26 (D4(GPIO2)), U3.6 (DC)
- net CS: now reaches U2.27 (D3(GPIO0)), U3.7 (CS)
- net SW: now reaches U2.30 (D0(GPIO16)), U5.3 (SW)
- net CLK: now reaches U2.4 (SD3(GPIO10)), U5.1 (CLK)
- net DT: now reaches U2.5 (SD2(GPIO9)), U5.2 (DT)
- net SCL L renamed SCL RTC
- net SDA L renamed SDA RTC
Other:
- moved on the sheet: BZ1, J1, R1, RV1, U2, U3, U4, U5

Commit message: esp01 minimal
Other:
- moved on the sheet: BZ1, J1, R1, RV1, U3, U4, U5

Commit message: new pcb
Connections:
- net +3V3: now also RV1.1; no longer RV1.3
- net GND: now also RV1.3; no longer RV1.1
Changed lines of the file:
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@@
     (pin "8")
   )
-  (symbol (lib_id "Device:R_Potentiometer") (at 58.42 127 0) (mirror x) (unit 1)
+  (symbol (lib_id "Device:R_Potentiometer") (at 58.42 127 0) (unit 1)
     (in_bom yes) (on_board yes) (fields_autoplaced)
     (property "Reference" "RV1" (id 0) (at 56.6421 126.1653 0)
