File: KiCad/espWatch-ESP01-minimal/espWatch-ESP01-minimal.kicad_sch (KiCad schematic)
At the start: 10 parts, among them J1 2-pin_power_input_header, SW1 SW_Push, U1 AMS1117-3.3, U2 ESP-01, U3 SSD1306_I2C_display, U4 DS3231_RTC_module

Commit message: esp01 minimal
Parts:
- added C3: 10u, My_Misc:CP_Radial_D5.0mm_P2.00mm_larger, symbol Device:C_Polarized
- added H1, H2, H3, H4: MountingHole, MountingHole:MountingHole_3.2mm_M3, symbol Mechanical:MountingHole
- added R3: 10k, My_Misc:R_Axial_DIN0207_L6.3mm_D2.5mm_P10.16mm_Horizontal_larger_pads, symbol Device:R
- added SW2: Function, My_Misc:SW_PUSH_6mm_large, symbol Switch:SW_Push
- SW1: value SW_Push -> Reset
- U2: footprint My_Arduino:ESP-01_w_pin_socket_large -> My_ESP8266:ESP-01_w_pin_socket_large
Connections:
- net +3V3: now also SW2.1
- net GND: now also C3.2, R3.1
- net VCC: now also C3.1
- net at U2.7 (GPIO3/UORxD): now also R3.2, SW2.2
